Commit message: add nvp meshes
Signed-off-by: wsribunm <worawissribunma@gmail.com>

File: nightvapor_description/urdf/nightvapor1.urdf (robot description, URDF)
Before this commit: robot nvp, 1 links, 0 joints
Links:
- removed link base_link
- added link nightvapor1; visual mesh filename=file:///home/wsribunm/ros2_ws/src/nightvapor/nightvapor_des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 scale=5 5 5

File: nightvapor_description/urdf/nightvapor2.urdf (robot description, URDF)
Before this commit: robot nvp, 1 links, 0 joints
Links:
- removed link base_link
- added link nightvapor2; visual mesh filename=file:///home/wsribunm/ros2_ws/src/nightvapor/nightvapor_des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 scale=5 5 5

File: nightvapor_description/urdf/nv1.urdf (robot description, URDF)
Before this commit: robot nvp, 1 links, 0 joints
Links:
- removed link base_link
- added link nv1; visual mesh filename=file:///home/wsribunm/ros2_ws/src/nightvapor/nightvapor_des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 scale=5 5 5
